Commit message: 20201008 git push after fork

File: wrs_gazebo/mobile_dual_arm/urdf/mobile_dual_arm.xacro (robot description, xacro)
@@ -10,4 +10,6 @@
   <xacro:include filename="$(find mobile_dual_arm)/urdf/mobile_dual_arm.gazebo" />
   <!--xacro:include filename="$(find mobile_table)/urdf/mobile_table.xacro" /-->
+  <xacro:include filename="$(find mobile_dual_arm)/urdf/shelf.xarco" />
+  <xacro:include filename="$(find mobile_dual_arm)/urdf/shelf1.xarco" />
   <link name="world"/>
   <joint name="fixed1" type="fixed">
@@ -28,4 +30,18 @@
     <parent link="mobile_base_footprint"/>
     <child link="base_link"/>
+  </joint>
+  <joint name="fixed_shelf1" type="fixed">
+      <!-- <origin
+       	xyz="-0.65 0.4625 -0.05"
+       	rpy="0 0 3.1416" /> -->
+    <parent link="world"/>
+    <child link="shelf_higher"/>
+  </joint>
+  <joint name="fixed_shelf2" type="fixed">
+    <!-- <origin
+      xyz="0.947 0.9 0 "
+     	rpy="0 0 1.5708" /> -->
+    <parent link="world"/>
+    <child link="shelf_higher2"/>
   </joint>
   <xacro:mir_100 prefix="mobile_"/>

File: wrs_gazebo/mobile_table/urdf/mobile_table.xacro (robot description, xacro)
@@ -1,2 +1,3 @@
+<?xml version="1.0"?>
 <robot
   name="mobile_table">

File: wrs_gazebo/single_arm/single_arm_description/urdf/single_arm.transmission.xacro (robot description, xacro)
@@ -72,4 +72,88 @@
     </actuator>
   </transmission>
+ <!-- <transmission name="${side}_tran1">
+    <type>transmission_interface/SimpleTransmission</type>
+    <joint name="${side}_joint_1">
+      <hardwareInterface>hardware_interface/PositionJointInterface</hardwareInterface>
+    </joint>
+    <actuator name="${side}_motor1">
+      <hardwareInterface>hardware_interface/PositionJointInterface</hardwareInterface>
+      <mechanicalReduction>1</mechanicalReduction>
+    </actuator>
+  </transmission>
+  <transmission name="${side}_tran2">
+    <type>transmission_interface/SimpleTransmission</type>
+    <joint name="${side}_joint_2">
+      <hardwareInterface>hardware_interface/PositionJointInterface</hardwareInterface>
+    </joint>
+    <actuator name="${side}_motor2">
+      <hardwareInterface>hardware_interface/PositionJointInterface</hardwareInterface>
+      <mechanicalReduction>1</mechanicalReduction>
+    </actuator>
+  </transmission>
+  <transmission name="${side}_tran3">
+    <type>transmission_interface/SimpleTransmission</type>
+    <joint name="${side}_joint_3">
+      <hardwareInterface>hardware_interface/PositionJointInterface</hardwareInterface>
+    </joint>
+    <actuator name="${side}_motor3">
+      <hardwareInterface>hardware_interface/PositionJointInterface</hardwareInterface>
+      <mechanicalReduction>1</mechanicalReduction>
+    </actuator>
+  </transmission>
+  <transmission name="${side}_tran4">
+    <type>transmission_interface/SimpleTransmission</type>
+    <joint name="${side}_joint_4">
+      <hardwareInterface>hardware_interface/PositionJointInterface</hardwareInterface>
+    </joint>
+    <actuator name="${side}_motor4">
+      <hardwareInterface>hardware_interface/PositionJointInterface</hardwareInterface>
+      <mechanicalReduction>1</mechanicalReduction>
+    </actuator>
+  </transmission>
+  <transmission name="${side}_tran5">
+    <type>transmission_interface/SimpleTransmission</type>
+    <joint name="${side}_joint_5">
+      <hardwareInterface>hardware_interface/PositionJointInterface</hardwareInterface>
+    </joint>
+    <actuator name="${side}_motor5">
+      <hardwareInterface>hardware_interface/PositionJointInterface</hardwareInterface>
+      <mechanicalReduction>1</mechanicalReduction>
+    </actuator>
+  </transmission>
+  <transmission name="${side}_tran6">
+    <type>transmission_interface/SimpleTransmission</type>
+    <joint name="${side}_joint_6">
+      <hardwareInterface>hardware_interface/PositionJointInterface</hardwareInterface>
+    </joint>
+    <actuator name="${side}_motor6">
+      <hardwareInterface>hardware_interface/PositionJointInterface</hardwareInterface>
+      <mechanicalReduction>1</mechanicalReduction>
+    </actuator>
+  </transmission>
+  <transmission name="${side}_tran7">
+    <type>transmission_interface/SimpleTransmission</type>
+    <joint name="${side}_joint_7">
+      <hardwareInterface>hardware_interface/PositionJointInterface</hardwareInterface>
+    </joint>
+    <actuator name="${side}_motor7">
+      <hardwareInterface>hardware_interface/PositionJointInterface</hardwareInterface>
+      <mechanicalReduction>1</mechanicalReduction>
+    </actuator>
+  </transmission> -->
 </xacro:macro>
+  <!-- <xacro:single_arm_transmission joint_name="r_joint_1"/>
+  <xacro:single_arm_transmission joint_name="r_joint_2"/>
+  <xacro:single_arm_transmission joint_name="r_joint_3"/>
+  <xacro:single_arm_transmission joint_name="r_joint_4"/>
+  <xacro:single_arm_transmission joint_name="r_joint_5"/>
+  <xacro:single_arm_transmission joint_name="r_joint_6"/>
+  <xacro:single_arm_transmission joint_name="r_joint_7"/>
+  <xacro:single_arm_transmission joint_name="l_jont_1"/>
+  <xacro:single_arm_transmission joint_name="l_jont_2"/>
+  <xacro:single_arm_transmission joint_name="l_jont_3"/>
+  <xacro:single_arm_transmission joint_name="l_jont_4"/>
+  <xacro:single_arm_transmission joint_name="l_jont_5"/>
+  <xacro:single_arm_transmission joint_name="l_jont_6"/>
+  <xacro:single_arm_transmission joint_name="l_jont_7"/> -->
 </robot>
