Commit message: fix dual_arm_notool but model jump in gazebo

File: wrs_gazebo/mobile_dual_arm/urdf/mobile_dual_arm_notool.xacro (robot description, xacro)
@@ -3,8 +3,8 @@
   <xacro:include filename="$(find mir_description)/urdf/include/mir_100_v1.urdf.xacro" />
   <!-- <xacro:include filename="$(find mir_description)/urdf/include/common.gazebo.xacro" /> -->
-  <xacro:include filename="$(find single_arm_description)/urdf/single_arm.xacro" />
+  <xacro:include filename="$(find single_arm_description)/urdf/single_arm_notool.xacro" />
   <xacro:include filename="$(find timda_body)/urdf/timda_body.xacro" />
   <!-- <xacro:include filename="$(find slide_rail)/urdf/slide_rail.xacro" /> -->
-  <xacro:include filename="$(find suction_urdf)/urdf/suction_urdf.xacro" />
+  <!--<xacro:include filename="$(find suction_urdf)/urdf/suction_urdf.xacro" />-->
   <!--xacro:include filename="$(find single_arm_description)/urdf/materials.xacro" /-->
   <xacro:include filename="$(find mobile_dual_arm)/urdf/mobile_dual_arm_notool.gazebo" />
@@ -46,5 +46,5 @@
   </joint>
   <xacro:mir_100 prefix="mobile_"/>
-  <xacro:single_arm side="r"  parent="slide_right" child="r_tool_link" toolrot="-1.57">
+  <!--<xacro:single_arm side="r"  parent="slide_right" child="r_tool_link" toolrot="-1.57">
     <origin xyz="0.0 0.1151 0.0" rpy="1.57 3.1415926 3.1415926" />
   </xacro:single_arm>
@@ -57,13 +57,13 @@
   <xacro:suction side="l"  parent="l_Link_6">
     <origin xyz="0 0.016 0" rpy="0 0 1.57" />
-  </xacro:suction>
-  <!-- <link name= "r_tool_link"/>
-  <xacro:single_arm side="r"  parent="slide_right" child="r_tool_link" toolrot="-1.57">
+  </xacro:suction>-->
+  <!-- <link name= "r_tool_link"/> -->
+  <!-- <link name= "l_tool_link"/> -->
+  <xacro:single_arm side="r"  parent="slide_right" child="" toolrot="-1.57">
     <origin xyz="0.0 0.1151 0.0" rpy="1.57 3.1415926 3.1415926" />
   </xacro:single_arm>
-  <link name= "l_tool_link"/>
-  <xacro:single_arm side="l"  parent="slide_left" child="l_tool_link" toolrot="1.57">
+  <xacro:single_arm side="l"  parent="slide_left" child="" toolrot="1.57">
     <origin xyz="0.0 0.1151 0.0" rpy="-1.57 0 0" />
-  </xacro:single_arm>  -->
+  </xacro:single_arm>
 <!--
   <joint name="fixed" type="fixed">
