Commit message: remove shelf1

File: wrs_gazebo/mobile_dual_arm/urdf/mobile_dual_arm_notoolend.xacro (robot description, xacro)
@@ -10,5 +10,5 @@
   <xacro:include filename="$(find mobile_dual_arm)/urdf/mobile_dual_arm.gazebo" />
   <!--xacro:include filename="$(find mobile_table)/urdf/mobile_table.xacro" /-->
-  <xacro:include filename="$(find mobile_dual_arm)/urdf/shelf.xarco" />
+  <!--<xacro:include filename="$(find mobile_dual_arm)/urdf/shelf.xarco" />-->
   <xacro:include filename="$(find mobile_dual_arm)/urdf/shelf1.xarco" />
   <link name="world"/>
@@ -31,11 +31,11 @@
     <child link="base_link"/>
   </joint>
-  <joint name="fixed_shelf1" type="fixed">
-      <!-- <origin
+  <!--<joint name="fixed_shelf1" type="fixed">
+      <origin
        	xyz="-0.65 0.4625 -0.05"
-       	rpy="0 0 3.1416" /> -->
+       	rpy="0 0 3.1416" />
     <parent link="world"/>
     <child link="shelf_higher"/>
-  </joint>
+  </joint>-->
   <joint name="fixed_shelf2" type="fixed">
     <!-- <origin
